Commit message: spawn robot

File: urdf/robot.urdf (robot description, URDF)
Before this commit: robot my-robot, 6 links, 5 joints
Joints:
- joint base_joint: origin xyz=0 0 0.31 rpy=0 0 0 -> xyz=0 0 0 rpy=0 0 0

Commit message: xong gmapping

File: urdf/robot.urdf (robot description, URDF)
Before this commit: robot my-robot, 6 links, 5 joints
Joints:
- joint lidar_joint: origin xyz=0 0 0.5 rpy=0 0 0 -> xyz=0 0 0.15 rpy=0 0 0

Commit message: fix navigation

File: urdf/robot.urdf (robot description, URDF)
Before this commit: robot my-robot, 6 links, 5 joints
Joints:
- joint lidar_joint: origin xyz=0 0 0.15 rpy=0 0 0 -> xyz=0 0 0.15 rpy=0 0 3.149159

Commit message: acml 1

File: urdf/robot.urdf (robot description, URDF)
Before this commit: robot my-robot, 6 links, 5 joints
Joints:
- joint lidar_joint: origin xyz=0 0 0.15 rpy=0 0 3.149159 -> xyz=0 0 0.15 rpy=0 0 3.14159

Commit message: sửa xong phần navigation

File: urdf/robot.urdf (robot description, URDF)
Before this commit: robot my-robot, 6 links, 5 joints
Joints:
- joint base_joint: origin xyz=0 0 0 rpy=0 0 0 -> xyz=0 0 0 rpy=0 0 -1.5708
- joint lidar_joint: origin xyz=0 0 0.15 rpy=0 0 3.14159 -> xyz=0 0 0.15 rpy=0 0 1.5708
